File: Hardware/OPA548_dev/opa548_0x00/opa548_0x00.kicad_pcb (KiCad board)
At the start: 2 copper layers, 160 x 59 mm, 25 parts, among them J3 Conn_01x03, J4 Conn_01x03, U1 OPA548FKTWT, U2 L7805, U3 INA226, U4 SC0915

Commit message: added ads
Parts:
- removed RV1: 10k, Potentiometer_THT:Potentiometer_Alpha_RD901F-40-00D_Single_Vertical_CircularHoles
- removed RV2: 20k, Potentiometer_THT:Potentiometer_Alpha_RD901F-40-00D_Single_Vertical_CircularHoles
- removed U4: SC0915, MyLib:MODULE_SC0915
- added C3: 1uF, Capacitor_SMD:C_1210_3225Metric, F.Cu at (181.0, 133.0)
- added C4: 1uF, Capacitor_SMD:C_1210_3225Metric, F.Cu at (155.5, 133.0)
- added FL1: Filter_EMI_CommonMode, MyLib:P0420NL, F.Cu at (175.6, 133.0)
- added HS1: Heatsink, Heatsink:Heatsink_38x38mm_SpringFixation, F.Cu at (7.89, 55.1)
- added J5: Conn_01x02, TerminalBlock:TerminalBlock_bornier-2_P5.08mm, F.Cu at (188.5, 135.5)
- added J6: Conn_01x08, Connector_PinHeader_2.00mm:PinHeader_1x08_P2.00mm_Vertical, F.Cu at (170.0, 106.0)
- moved R1 67.3 mm to (140.0, 111.2)
- moved R3 67.3 mm to (140.0, 117.0)
- moved R4 67.3 mm to (140.0, 120.0)
- moved R2 67.3 mm to (140.0, 114.1)
- moved R7 60.5 mm to (134.2, 114.4)
- moved R5 60.5 mm to (134.2, 111.5)
- moved R8 60.5 mm to (134.2, 117.3)
- moved R9 60.5 mm to (134.2, 120.3)
- moved H1 60.0 mm to (190.0, 100.0)
- moved H2 60.0 mm to (190.0, 149.0)
- moved U2 43.3 mm to (124.7, 115.4)
- moved U1 40.0 mm to (142.2, 143.1), turned to -90 degrees
- moved U3 13.2 mm to (128.5, 127.0), turned to -90 degrees
- moved R6 1.38 mm to (128.5, 133.2), turned to 90 degrees
Connections:
- net Net-(J3-Pin_2) renamed /VLim_set
- net Net-(J4-Pin_2) renamed /ILim_set
- R6 pad 1: Net-(U1-Vo) -> Net-(J1-Pad1)
- R6 pad 2: Net-(U3-Vin+) -> Net-(U3-Vin-)
- R6 pad 3: Net-(U3-Vin-) -> Net-(U3-Vin+)
- R6 pad 4: Net-(J1-Pad1) -> Net-(U1-Vo)
- U1 pad 8: (no net) -> unconnected-(U1-EP-Pad8)
Routing:
- net Net-(U1-Vo): track 0.00 -> 8.36 mm
- net GND: track 0.00 -> 3.97 mm, vias 0 -> 2
- net Net-(U3-Vin-): track 0.00 -> 3.44 mm
- net /VLim_set: track 0.00 -> 3.25 mm, vias 0 -> 1
- net Net-(U1-Vin-): track 0.00 -> 3.24 mm, vias 0 -> 1
- net /ILim_set: track 0.00 -> 3.23 mm, vias 0 -> 1
- net Net-(U3-Vin+): track 0.00 -> 2.76 mm
- net unconnected-(U1-EP-Pad8): vias 0 -> 91
- added copper zone on B.Cu, net GND
- added copper zone on F.Cu, net Net-(J1-Pad1)
- added copper zone on F.Cu, net Net-(J5-Pin_1)
- added copper zone on F.Cu, net Net-(J5-Pin_2)
- added copper zone on F.Cu, net Net-(U1-Vo)
- added copper zone on F.Cu, net VCC
- added copper zone on B.Cu, net unconnected-(U1-EP-Pad8)
- added copper zone on F.Cu, net unconnected-(U1-EP-Pad8)
Other:
- board size 160 x 59 mm -> 100 x 59 mm
