File: Hardware/OPA548_dev/opa548_0x00/opa548_0x00.kicad_sch (KiCad schematic)
At the start: 25 parts, among them J3 Conn_01x03, J4 Conn_01x03, U1 OPA548FKTWT, U2 L7805, U3 INA226, U4 SC0915

Commit message: added ads
Parts:
- removed U4: SC0915, MyLib:MODULE_SC0915, symbol MyLib:SC0915
- added C3, C4: 1uF, Capacitor_SMD:C_1210_3225Metric, symbol Device:C_Small
- added FL1: Filter_EMI_CommonMode, MyLib:P0420NL, symbol Device:Filter_EMI_CommonMode
- added HS1: Heatsink, Heatsink:Heatsink_38x38mm_SpringFixation, symbol Mechanical:Heatsink
- added J5: Conn_01x02, TerminalBlock:TerminalBlock_bornier-2_P5.08mm, symbol Connector_Generic:Conn_01x02
- added J6: Conn_01x08, Connector_PinHeader_2.00mm:PinHeader_1x08_P2.00mm_Vertical, symbol Connector_Generic:Conn_01x08
- RV1, RV2: now not fitted
Connections:
- net +3.3V: now also J6.1 (Pin_1)
- net +5V: now also J6.2 (Pin_2)
- net Alert: now also J6.7 (Pin_7)
- net GND: now also C4.2, FL1.2, J6.8 (Pin_8)
- net SCL: now also J6.6 (Pin_6)
- net SDA: now also J6.5 (Pin_5)
- net VCC: now also C4.1, FL1.4
- net VLim_set: now reaches J3.2 (Pin_2), RV1.2, U1.1 (Vin+)
- net VLim_set: now also J6.4 (Pin_4)
- net ILim_set: now reaches C1.1, J4.2 (Pin_2), RV2.2, U1.3 (Ilim)
- net ILim_set: now also J6.3 (Pin_3)
- net at R1.2, U1.6 (Vo), U3.8 (Vbus): now also R6.4; no longer R6.1
- net at R6.2: now also U3.9 (Vin-); no longer U3.10 (Vin+)
- net at R6.3: now also U3.10 (Vin+); no longer U3.9 (Vin-)
- net at J1.1: now also R6.1; no longer R6.4
- new net: C3.1, FL1.3, J5.1 (Pin_1)
- new net: C3.2, FL1.1, J5.2 (Pin_2)
Other:
- moved on the sheet: H1, H2, H3, H4, R6, U2
